Commit message: Commit

File: robot/ros2_ws/src/my_robot_description/urdf/my_robot.urdf.xacro (robot description, xacro)
@@ -66,5 +66,5 @@
                        origin_y="${-0.235-(wheel_length/2.0)*cos(pi/3)}"
                        axis="${sin(pi/6)} ${cos(pi/6)} 0"/>
-    <link name="lidar">
+    <link name="laser">
         <visual>
             <geometry>
@@ -74,8 +74,8 @@
         </visual>
     </link>
-    <joint name="lidar_to_upper_body_joint" type="fixed">
+    <joint name="laserr_to_upper_body_joint" type="fixed">
         <parent link="upper_body"/>
-        <child link="lidar"/>
-        <origin xyz="0 0 0.265" roy="0 0 0"/>
+        <child link="laser"/>
+        <origin xyz="0 0 0.265" rpy="0 0 0"/>
     </joint>
 </robot>

Commit message: H

File: robot/ros2_ws/src/my_robot_description/urdf/my_robot.urdf.xacro (robot description, xacro)
@@ -22,5 +22,5 @@
     <link name="upper_body">
         <visual>
-            <origin xyz="0 0 0" rpy ="0 0 0.5216"/>
+            <origin xyz="0 0 0" rpy ="0 0 -0.5216"/>
             <geometry>
                 <mesh filename="package://my_robot_description/meshes/upper_body.stl" scale="0.001 0.001 0.001"/>

Commit message: HELP

File: robot/ros2_ws/src/my_robot_description/urdf/my_robot.urdf.xacro (robot description, xacro)
@@ -22,5 +22,5 @@
     <link name="upper_body">
         <visual>
-            <origin xyz="0 0 0" rpy ="0 0 -0.5216"/>
+            <origin xyz="0 0 0" rpy ="0 0 0.5216"/>
             <geometry>
                 <mesh filename="package://my_robot_description/meshes/upper_body.stl" scale="0.001 0.001 0.001"/>
@@ -66,5 +66,5 @@
                        origin_y="${-0.235-(wheel_length/2.0)*cos(pi/3)}"
                        axis="${sin(pi/6)} ${cos(pi/6)} 0"/>
-    <link name="laser">
+    <link name="lidar">
         <visual>
             <geometry>
@@ -74,8 +74,8 @@
         </visual>
     </link>
-    <joint name="laserr_to_upper_body_joint" type="fixed">
+    <joint name="lidar_to_upper_body_joint" type="fixed">
         <parent link="upper_body"/>
-        <child link="laser"/>
-        <origin xyz="0 0 0.265" rpy="0 0 0"/>
+        <child link="lidar"/>
+        <origin xyz="0 0 0.265" roy="0 0 0"/>
     </joint>
 </robot>
