Commit message: GOT DA FKIN LIDAR WORKING LESGOOOOOOgit add .git add .!

File: robot/ros2_ws/install/my_robot_description/share/my_robot_description/urdf/my_robot.urdf.xacro (robot description, xacro)
@@ -74,8 +74,8 @@
         </visual>
     </link>
-    <joint name="laserr_to_upper_body_joint" type="fixed">
+    <joint name="laser_to_upper_body_joint" type="fixed">
         <parent link="upper_body"/>
         <child link="laser"/>
-        <origin xyz="0 0 0.265" rpy="0 0 0"/>
+        <origin xyz="0 0 0.265" roy="0 0 0"/>
     </joint>
 </robot>

File: robot/ros2_ws/src/my_robot_description/urdf/my_robot.urdf.xacro (robot description, xacro)
@@ -66,5 +66,5 @@
                        origin_y="${-0.235-(wheel_length/2.0)*cos(pi/3)}"
                        axis="${sin(pi/6)} ${cos(pi/6)} 0"/>
-    <link name="lidar">
+    <link name="laser">
         <visual>
             <geometry>
@@ -74,7 +74,7 @@
         </visual>
     </link>
-    <joint name="lidar_to_upper_body_joint" type="fixed">
+    <joint name="laser_to_upper_body_joint" type="fixed">
         <parent link="upper_body"/>
-        <child link="lidar"/>
+        <child link="laser"/>
         <origin xyz="0 0 0.265" roy="0 0 0"/>
     </joint>

Commit message: Working

File: robot/ros2_ws/install/my_robot_description/share/my_robot_description/urdf/my_robot.urdf.xacro (robot description, xacro)
@@ -77,5 +77,5 @@
         <parent link="upper_body"/>
         <child link="laser"/>
-        <origin xyz="0 0 0.265" roy="0 0 0"/>
+        <origin xyz="0 0 0.265" rpy="0 0 0"/>
     </joint>
 </robot>
