Commit message: Fixed arduino odom issue

File: install/my_robot_description/share/my_robot_description/urdf/my_robot.urdf.xacro (robot description, xacro)
@@ -26,4 +26,5 @@
                 <mesh filename="package://my_robot_description/meshes/upper_body.stl" scale="0.001 0.001 0.001"/>
             </geometry>
+            <material name="pink"/>
         </visual>
     </link>
@@ -65,5 +66,5 @@
                        origin_y="${-0.235-(wheel_length/2.0)*cos(pi/3)}"
                        axis="${sin(pi/6)} ${cos(pi/6)} 0"/>
-    <link name="lidar">
+    <link name="laser">
         <visual>
             <geometry>
@@ -73,8 +74,8 @@
         </visual>
     </link>
-    <joint name="lidar_to_upper_body_joint" type="fixed">
+    <joint name="laser_to_upper_body_joint" type="fixed">
         <parent link="upper_body"/>
-        <child link="lidar"/>
-        <origin xyz="0 0 0.265" roy="0 0 0"/>
+        <child link="laser"/>
+        <origin xyz="0 0 0.265" rpy="0 0 0"/>
     </joint>
 </robot>
